File: astrobox_control/pwmcontrolplane.kicad_sch (KiCad schematic)
At the start: 26 parts, among them J6 Fader_PWM1, J7 Fader_PWM2, J8 Fader_PWM3, J9 ISP_PWM_Driver, U6 ATmega644-20P, U7 L298N, U8 L298N, U9 DHT11

Commit message: astrobox WIP
Parts:
- added C44: 100n, Capacitor_SMD:C_1206_3216Metric_Pad1.33x1.80mm_HandSolder, symbol Device:C
- added U19: 24LC16, Package_DIP:DIP-8_W7.62mm, symbol Memory_EEPROM:24LC16
Connections:
- net +5V: now also C44.1, U19.8 (VCC)
- net GND: now also C44.2, U19.1 (A0), U19.2 (A1), U19.3 (A2), U19.4 (GND), U19.7 (WP)
- net SCL: now also U19.6 (SCL)
- net SDA: now also U19.5 (SDA)
