File: astrobox_power/Internal_Bat_Subsystem.kicad_sch (KiCad schematic)
At the start: 18 parts, among them Q3 IRLZ34N, SW5 SW_PWR_ON, U2 L7812, U3 L7805, U4 ATtiny85-20P, U5 DHT11

Commit message: astrobox WIP
Parts:
- added J11: ISP, Connector_PinHeader_2.54mm:PinHeader_2x03_P2.54mm_Vertical, symbol Connector_Generic:Conn_02x03_Odd_Even
Connections:
- net SCL: now also J11.1 (Pin_1)
- net SDA: now also J11.5 (Pin_5)
- net GND: now reaches BT2.2 (-), C10.1, C11.2, C12.1, C13.2, C9.2, Q3.3 (S), R5.1, R6.1, R7.2, U2.2 (GND), U3.2 (GND), U4.4 (GND), U5.4 (GND)
- net GND: now also J11.4 (Pin_4)
- net at D8.2 (A), Q3.1 (G), R5.2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: now also J11.3 (Pin_3)
- net at C11.1, C13.1, U3.3 (OUT)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: now also J11.6 (Pin_6)
- net at U4.1 (~{RESET}/PB5), U5.2 (IO): now also J11.2 (Pin_2)
Other:
- title: (none) -> Astrobox 
