File: astrobox_power/StepUp_15V.kicad_sch (KiCad schematic)
At the start: 13 parts, among them Q2 BUZ11, U1 MC34063AP

Commit message: astrobox WIP
Parts:
- R2: footprint Resistor_THT:R_Axial_Power_L20.0mm_W6.4mm_P22.40mm -> Resistor_THT:R_Axial_DIN0207_L6.3mm_D2.5mm_P10.16mm_Horizontal
Other:
- title: (none) -> Astrobox 
Changed lines of the file:
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@@
 	(generator_version "8.0")
 	(paper "A4")
+	(title_block
+		(title "Astrobox ")
+		(date "2024-05-01")
+		(rev "3")
+		(comment 1 "Napajeci modul")
+	)
 	(junction
 		(at 101.6 61.595)
@@
 			)
 		)
-		(property "Footprint" "Resistor_THT:R_Axial_Power_L20.0mm_W6.4mm_P22.40mm"
+		(property "Footprint" "Resistor_THT:R_Axial_DIN0207_L6.3mm_D2.5mm_P10.16mm_Horizontal"
 			(at 114.935 63.373 90)
 			(effects
