File: astrobox_power/astrobox_power.kicad_sch (KiCad schematic)
At the start: 40 parts, among them J1 IEC C14 POWER IN, J10 FAN_AUTO, J2 Zas1, J3 Zas2, J4 Zas3, J5 Zas4, J6 INTERCOM1, J7 POWER_OUT, J8 PWR_IN, J9 PWR_IN_BAT, K1 G5LE-1, K2 G5LE-1, K3 G5LE-1, K4 G5LE-1, Q1 IRF4905, Q4 IRLZ34N, SW1 PWR_OUT_1, SW2 PWR_OUT_2, SW3 PWR_OUT_3, SW4 PWR_OUT_4, U6 4N25

Commit message: astrobox WIP
Other:
- title: Astrobox -> Astrobox 
Changed lines of the file:
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@@
 	(paper "A4")
 	(title_block
-		(title "Astrobox")
-		(date "2024-04-13")
-		(rev "2")
+		(title "Astrobox ")
+		(date "2024-05-01")
+		(rev "3")
+		(comment 1 "Napajeci modul")
 	)
 	(junction
