File: astrobox_radio_input/astrobox_radio_input.kicad_pcb (KiCad board)
At the start: 2 copper layers, 100 x 108 mm, 25 parts, among them J1 Satelite finder, J2 GPS Modul GY-NEO6MV2, J3 INTERCOM1, J4 ADS1115 modul, J5 EXT_PWR, J6 INTERCOM2, J7 I2C, J8 Raspberry_Pi, U1 L7805, U2 L7805

Commit message: astrobox WIP
Parts:
- removed the REF** at (69.3, 126.1)
- removed the REF** at (69.3, 77.1)
- removed the REF** at (127.3, 126.1)
- removed the REF** at (127.3, 77.1)
- added REF**: KiCad-Logo2_5mm_SilkScreen, Symbol:KiCad-Logo2_5mm_SilkScreen, F.Cu at (75.6, 77.9)
- added REF**: OSHW-Logo2_7.3x6mm_SilkScreen, Symbol:OSHW-Logo2_7.3x6mm_SilkScreen, F.Cu at (86.0, 78.3)
- moved REF** 55.0 mm to (155.0, 78.0)
- moved REF** 55.0 mm to (65.0, 78.0)
- moved J5 32.3 mm to (129.9, 74.7), turned to -90 degrees
- moved J7 15.9 mm to (144.9, 74.7), turned to -90 degrees
Routing:
- net /5V: track 122.0 -> 98.5 mm
- net /SCL: track 174.3 -> 166.6 mm
- net /SDA: track 172.1 -> 169.5 mm
Other:
- board size 100 x 108 mm -> 99.9 x 52.9 mm
- board text added: "Astrobox radio input module"
- board text added: "GND +5V"
- board text added: "SCL SDA"
- board text added: "https://github.com/SniperCZE/astrobox"
- board text removed: "GND SDA +5V SCL"
