File: astrobox_medium/astrobox_power_mediumbox/_autosave-astrobox_power_mediumbox.kicad_pcb (KiCad board)
At the start: 2 copper layers, 73.5 x 91.5 mm, 310 parts, among them J1 OUT_12V_1, J10 OUT_5V, J11 OUT_6V, J12 OUT_9V, J13 ISP, J14 TO_CONTROL, J15 TO_OUTPUT, J2 OUT_12V_2, J3 OUT_12V_3, J4 OUT_12V_4, J5 OUT_12V_5, J6 OUT_12V_6, J7 OUT_12V_7, J8 OUT_12V_8, J9 POWER_IN, Q1 BC807, Q10 BC817, Q11 BC817, Q12 BC817, Q13 BC817, Q14 BC817, Q15 BC817, Q16 BC817, Q17 IRLZ34N, Q18 IRLZ34N, Q19 IRLZ34N, Q2 BC807, Q20 IRLZ34N, Q21 IRLZ34N, Q22 IRLZ34N, Q23 IRLZ34N, Q24 IRLZ34N, Q25 BC807, Q26 BC807, Q27 BC807, Q28 BC807, Q29 BC807, Q3 BC807, Q30 BC807, Q31 BC807, Q33 BC817, Q34 BC817, Q35 BC817, Q36 BC817, Q37 BC817, Q38 BC817, Q39 BC817, Q4 BC807, Q40 BC817, Q41 IRLZ34N, Q42 IRLZ34N, Q43 IRLZ34N, Q44 BC807, Q5 BC807, Q6 BC807, Q7 BC807, Q8 BC807, Q9 BC817, SW1 PWM_ENB_1, SW10 ENB_9V, SW11 ENB_12V_6, SW12 ENB_6V, SW13 ENB_12V_5, SW14 ENB_5V, SW15 ENB_12V_4, SW16 PWM_ENB_5, SW17 PWM_ENB_6, SW18 PWM_ENB_7, SW19 PWM_ENB_8, SW2 PWM_ENB_2, SW3 PWM_ENB_3, SW4 PWM_ENB_4, SW5 ENB_12V_3, SW6 ENB_12V_2, SW7 ENB_12V_8, SW8 ENB_12V_1, SW9 ENB_12V_7, U1 DA56-11EWA, U10 NE555P, U11 NE555P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

Commit message: medium astrobox in multiple boards
Parts:
- removed J14: TO_CONTROL, Connector_PinHeader_2.54mm:PinHeader_1x29_P2.54mm_Vertical
- removed J15: TO_OUTPUT, Connector_PinHeader_2.54mm:PinHeader_1x29_P2.54mm_Vertical
- removed Q43: IRLZ34N, Package_TO_SOT_THT:TO-220-3_Vertical
- added Q32: IRLR024NTRPBF, Package_TO_SOT_SMD:TO-252-3_TabPin2, F.Cu at (386.0, 90.3)
- added REF**: MountingHole_3.2mm_M3_Pad_Via, MountingHole:MountingHole_3.2mm_M3_Pad_Via, F.Cu at (267.5, 26.2)
- added REF**: MountingHole_3.2mm_M3_Pad_Via, MountingHole:MountingHole_3.2mm_M3_Pad_Via, F.Cu at (265.9, 139.2)
- added REF**: MountingHole_3.2mm_M3_Pad_Via, MountingHole:MountingHole_3.2mm_M3_Pad_Via, F.Cu at (91.7, 84.3)
- added REF**: MountingHole_3.2mm_M3_Pad_Via, MountingHole:MountingHole_3.2mm_M3_Pad_Via, F.Cu at (25.7, 150.4)
- added REF**: MountingHole_3.2mm_M3_Pad_Via, MountingHole:MountingHole_3.2mm_M3_Pad_Via, F.Cu at (24.9, 24.6)
- added REF**: MountingHole_3.2mm_M3_Pad_Via, MountingHole:MountingHole_3.2mm_M3_Pad_Via, F.Cu at (149.7, 27.3)
- added REF**: MountingHole_3.2mm_M3_Pad_Via, MountingHole:MountingHole_3.2mm_M3_Pad_Via, F.Cu at (211.8, 85.6)
- added REF**: MountingHole_3.2mm_M3_Pad_Via, MountingHole:MountingHole_3.2mm_M3_Pad_Via, F.Cu at (149.1, 143.8)
- Q17, Q18, Q19, Q20, Q21, Q22, Q23, Q24, Q41, Q42: value IRLZ34N -> IRLR024NTRPBF; footprint Package_TO_SOT_THT:TO-220-3_Vertical -> Package_TO_SOT_SMD:TO-252-3_TabPin2
- moved SW7 411.8 mm to (395.6, 301.3)
- moved SW9 401.4 mm to (375.0, 301.5)
- moved SW6 385.4 mm to (394.9, 246.8)
- moved SW11 382.4 mm to (358.6, 301.2)
- moved SW8 366.1 mm to (369.9, 244.7)
- moved SW13 364.1 mm to (342.8, 301.0)
- moved D19 363.5 mm to (397.8, 312.7)
- moved SW15 356.3 mm to (320.8, 300.1)
- moved R114 353.3 mm to (-102.4, 231.4)
- moved R115 353.3 mm to (-102.4, 234.8)
- moved R53 347.4 mm to (-104.4, 251.5)
- moved R41 344.8 mm to (-116.9, 250.0)
- moved SW10 341.4 mm to (346.5, 244.9)
- moved SW5 341.1 mm to (298.1, 299.4)
- moved R89 339.5 mm to (393.4, 287.5)
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Connections:
- Q41 pad 2: Net-(J10-Pin_1) -> GND
- Q41 pad 3: GND -> Net-(J10-Pin_1)
- Q42 pad 2: Net-(J11-Pin_1) -> GND
- Q42 pad 3: GND -> Net-(J12-Pin_1)
- R58 pad 1: Net-(Q42-G) -> Net-(Q32-G)
- R59 pad 1: Net-(Q43-G) -> Net-(Q42-G)
- R65 pad 2: Net-(Q42-G) -> Net-(Q32-G)
- R66 pad 2: Net-(Q43-G) -> Net-(Q42-G)
Other:
- board size 73.5 x 91.5 mm -> 524.9 x 233.1 mm
