File: astrobox_medium/astrobox_power_mediumbox/astrobox_power_mediumbox.kicad_pcb (KiCad board)
At the start: 2 copper layers, 260 x 140 mm, 316 parts, among them J1 OUT_12V_1, J10 OUT_5V, J11 OUT_6V, J12 OUT_9V, J13 ISP, J2 OUT_12V_2, J3 OUT_12V_3, J4 OUT_12V_4, J5 OUT_12V_5, J6 OUT_12V_6, J7 OUT_12V_7, J8 OUT_12V_8, J9 POWER_IN, Q1 BC807, Q10 BC817, Q11 BC817, Q12 BC817, Q13 BC817, Q14 BC817, Q15 BC817, Q16 BC817, Q17 IRLR024NTRPBF, Q18 IRLR024NTRPBF, Q19 IRLR024NTRPBF, Q2 BC807, Q20 IRLR024NTRPBF, Q21 IRLR024NTRPBF, Q22 IRLR024NTRPBF, Q23 IRLR024NTRPBF, Q24 IRLR024NTRPBF, Q25 BC807, Q26 BC807, Q27 BC807, Q28 BC807, Q29 BC807, Q3 BC807, Q30 BC807, Q31 BC807, Q32 IRLR024NTRPBF, Q33 BC817, Q34 BC817, Q35 BC817, Q36 BC817, Q37 BC817, Q38 BC817, Q39 BC817, Q4 BC807, Q40 BC817, Q41 IRLR024NTRPBF, Q42 IRLR024NTRPBF, Q44 BC807, Q5 BC807, Q6 BC807, Q7 BC807, Q8 BC807, Q9 BC817, SW1 PWM_ENB_1, SW10 ENB_9V, SW11 ENB_12V_6, SW12 ENB_6V, SW13 ENB_12V_5, SW14 ENB_5V, SW15 ENB_12V_4, SW16 PWM_ENB_5, SW17 PWM_ENB_6, SW18 PWM_ENB_7, SW19 PWM_ENB_8, SW2 PWM_ENB_2, SW3 PWM_ENB_3, SW4 PWM_ENB_4, SW5 ENB_12V_3, SW6 ENB_12V_2, SW7 ENB_12V_8, SW8 ENB_12V_1, SW9 ENB_12V_7, U1 DA56-11EWA, U10 NE555P, U11 NE555P, U12 74LS08, U13 74LS08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

Commit message: astrobox medium final pcb
Parts:
- removed C1, C11, C13, C14, C15, C16, C17, C18, C19, C2, C20, C21, C22, C23, C24, C25, C26, C27, C28, C29, C3, C31, C33, C35, C37, C38, C39, C4, C5, C7, C9: 100n, Capacitor_SMD:C_1206_3216Metric_Pad1.33x1.80mm_HandSolder
- removed C10, C12, C30, C32, C34, C36, C6, C8: 1n, Capacitor_SMD:C_1206_3216Metric_Pad1.33x1.80mm_HandSolder
- removed D1, D14, D15, D16, D17, D2, D20, D21, D22, D23, D3, D4, D5, D6, D7, D8: 1N4007, Diode_SMD:D_SMA-SMB_Universal_Handsoldering
- removed D10: PWM_ENB_2, LED_THT:LED_D5.0mm
- removed D11: PWM_ENB_3, LED_THT:LED_D5.0mm
- removed D12: PWM_ENB_4, LED_THT:LED_D5.0mm
- removed D13: ENB_12V_3, LED_THT:LED_D5.0mm
- removed D18: ENB_12V_2, LED_THT:LED_D5.0mm
- removed D19: ENB_12V_8, LED_THT:LED_D5.0mm
- removed D24: ENB_12V_1, LED_THT:LED_D5.0mm
- removed D25: ENB_12V_7, LED_THT:LED_D5.0mm
- removed D26: ENB_9V, LED_THT:LED_D5.0mm
- removed D27: ENB_12V_6, LED_THT:LED_D5.0mm
- removed D28: ENB_6V, LED_THT:LED_D5.0mm
- removed D29: ENB_12V_5, LED_THT:LED_D5.0mm
- removed D30: ENB_5V, LED_THT:LED_D5.0mm
- removed D31: ENB_12V_4, LED_THT:LED_D5.0mm
- removed D32: PWM_ENB_5, LED_THT:LED_D5.0mm
- removed D33: PWM_ENB_6, LED_THT:LED_D5.0mm
- removed D34: PWM_ENB_7, LED_THT:LED_D5.0mm
- removed D35: PWM_ENB_8, LED_THT:LED_D5.0mm
- removed D9: PWM_ENB_1, LED_THT:LED_D5.0mm
- removed Q12, Q13, Q14, Q15, Q16, Q33, Q34, Q35, Q36, Q37, Q38, Q39, Q40: BC817, Package_TO_SOT_SMD:SOT-23_Handsoldering
- removed Q17, Q18, Q19, Q20, Q21, Q22, Q23, Q24, Q32, Q41, Q42: IRLR024NTRPBF, Package_TO_SOT_SMD:TO-252-3_TabPin2
- removed Q25, Q26, Q27, Q28, Q29, Q30, Q31, Q44: BC807, Package_TO_SOT_SMD:SOT-23_Handsoldering
- removed R100, R101, R102, R103, R104, R105, R67, R68, R69, R70, R71, R72, R73, R74, R75, R76, R77, R78, R87, R88, R89, R90, R91, R96, R97, R98, R99: 330R, Resistor_SMD:R_1206_3216Metric_Pad1.30x1.75mm_HandSolder
- removed R106, R107, R108, R109, R110, R111, R112, R113, R114, R115, R116, R117, R118, R119, R120, R121: 100k, Resistor_SMD:R_1206_3216Metric_Pad1.30x1.75mm_HandSolder
- removed R23, R24, R25, R26, R27, R28, R29, R57, R58, R59: 4k7, Resistor_SMD:R_1206_3216Metric_Pad1.30x1.75mm_HandSolder
- removed R30, R79, R80, R82, R84: 33R, Resistor_SMD:R_1206_3216Metric_Pad1.30x1.75mm_HandSolder
- removed R31, R32, R41, R42, R43, R44, R45, R46, R47, R48, R49, R50, R51, R52, R53, R54, R55, R56, R60, R61, R62, R63, R81, R83, R85, R86, R92, R93, R94, R95: 1k, Resistor_SMD:R_1206_3216Metric_Pad1.30x1.75mm_HandSolder
- removed R33, R34, R35, R36, R37, R38, R39, R40, R64, R65, R66: 470R, Resistor_SMD:R_1206_3216Metric_Pad1.30x1.75mm_HandSolder
- removed the REF** at (267.5, 26.2)
- removed the REF** at (265.9, 139.2)
- removed the REF** at (91.7, 84.3)
- removed the REF** at (25.7, 150.4)
- removed the REF** at (24.9, 24.6)
- removed the REF** at (149.7, 27.3)
- removed the REF** at (211.8, 85.6)
- removed the REF** at (149.1, 143.8)
- removed RV1: PWM_SET_1, Connector_Wire:SolderWire-1sqmm_1x03_P5.4mm_D1.4mm_OD2.7mm
- removed RV2: PWM_SET_2, Connector_Wire:SolderWire-1sqmm_1x03_P5.4mm_D1.4mm_OD2.7mm
- removed RV3: PWM_SET_3, Connector_Wire:SolderWire-1sqmm_1x03_P5.4mm_D1.4mm_OD2.7mm
- removed RV4: PWM_SET_4, Connector_Wire:SolderWire-1sqmm_1x03_P5.4mm_D1.4mm_OD2.7mm
- removed RV5: PWM_SET_5, Connector_Wire:SolderWire-1sqmm_1x03_P5.4mm_D1.4mm_OD2.7mm
- removed RV6: PWM_SET_6, Connector_Wire:SolderWire-1sqmm_1x03_P5.4mm_D1.4mm_OD2.7mm
- removed RV7: PWM_SET_7, Connector_Wire:SolderWire-1sqmm_1x03_P5.4mm_D1.4mm_OD2.7mm
- removed RV8: PWM_SET_8, Connector_Wire:SolderWire-1sqmm_1x03_P5.4mm_D1.4mm_OD2.7mm
- removed SW1: PWM_ENB_1, Connector_Wire:SolderWire-1sqmm_1x02_P5.4mm_D1.4mm_OD2.7mm
- removed SW10: ENB_9V, Connector_Wire:SolderWire-1sqmm_1x02_P5.4mm_D1.4mm_OD2.7mm
- removed SW11: ENB_12V_6, Connector_Wire:SolderWire-1sqmm_1x02_P5.4mm_D1.4mm_OD2.7mm
- removed SW12: ENB_6V, Connector_Wire:SolderWire-1sqmm_1x02_P5.4mm_D1.4mm_OD2.7mm
- removed SW13: ENB_12V_5, Connector_Wire:SolderWire-1sqmm_1x02_P5.4mm_D1.4mm_OD2.7mm
- removed SW14: ENB_5V, Connector_Wire:SolderWire-1sqmm_1x02_P5.4mm_D1.4mm_OD2.7mm
- removed SW15: ENB_12V_4, Connector_Wire:SolderWire-1sqmm_1x02_P5.4mm_D1.4mm_OD2.7mm
- removed SW16: PWM_ENB_5, Connector_Wire:SolderWire-1sqmm_1x02_P5.4mm_D1.4mm_OD2.7mm
- removed SW17: PWM_ENB_6, Connector_Wire:SolderWire-1sqmm_1x02_P5.4mm_D1.4mm_OD2.7mm
- removed SW18: PWM_ENB_7, Connector_Wire:SolderWire-1sqmm_1x02_P5.4mm_D1.4mm_OD2.7mm
- removed SW19: PWM_ENB_8, Connector_Wire:SolderWire-1sqmm_1x02_P5.4mm_D1.4mm_OD2.7mm
- removed SW2: PWM_ENB_2, Connector_Wire:SolderWire-1sqmm_1x02_P5.4mm_D1.4mm_OD2.7mm
- removed SW3: PWM_ENB_3, Connector_Wire:SolderWire-1sqmm_1x02_P5.4mm_D1.4mm_OD2.7mm
- removed SW4: PWM_ENB_4, Connector_Wire:SolderWire-1sqmm_1x02_P5.4mm_D1.4mm_OD2.7mm
- removed SW5: ENB_12V_3, Connector_Wire:SolderWire-1sqmm_1x02_P5.4mm_D1.4mm_OD2.7mm
- removed SW6: ENB_12V_2, Connector_Wire:SolderWire-1sqmm_1x02_P5.4mm_D1.4mm_OD2.7mm
- removed SW7: ENB_12V_8, Connector_Wire:SolderWire-1sqmm_1x02_P5.4mm_D1.4mm_OD2.7mm
- removed SW8: ENB_12V_1, Connector_Wire:SolderWire-1sqmm_1x02_P5.4mm_D1.4mm_OD2.7mm
- removed SW9: ENB_12V_7, Connector_Wire:SolderWire-1sqmm_1x02_P5.4mm_D1.4mm_OD2.7mm
- removed U1, U2, U3, U4, U5, U6, U7, U8: DA56-11EWA, Display_7Segment:DA56-11SURKWA
- removed U10, U11, U14, U23, U24, U25, U26, U9: NE555P, Package_SO:SOIC-8_5.3x6.2mm_P1.27mm
- removed U12, U13, U20, U22, U27, U30: 74LS08, Package_SO:SO-14_3.9x8.65mm_P1.27mm
- removed U15, U16: 74LS32, Package_DIP:DIP-14_W7.62mm_Socket
- removed U17, U18: 74AHC04, Package_SO:SO-14_3.9x8.65mm_P1.27mm
- removed U19: 74LS47, Package_DIP:DIP-16_W7.62mm_Socket
- removed U21, U29: 74HC4051, Package_SO:SOIC-16_3.9x9.9mm_P1.27mm
- removed U28: ATmega16A-M, Package_QFP:TQFP-44-1EP_10x10mm_P0.8mm_EP4.5x4.5mm
- added ?: , , F.Cu at (77.2, 94.9)
- added J14: +5V, Connector_PinHeader_2.54mm:PinHeader_1x11_P2.54mm_Vertical, F.Cu at (73.2, 86.8)
- added J15: Control, Connector_PinHeader_2.54mm:PinHeader_1x11_P2.54mm_Vertical, F.Cu at (134.7, 86.9)
- added REF**: MountingHole_3.2mm_M3_Pad_Via, MountingHole:MountingHole_3.2mm_M3_Pad_Via, F.Cu at (155.0, 45.0)
- added REF**: MountingHole_3.2mm_M3_Pad_Via, MountingHole:MountingHole_3.2mm_M3_Pad_Via, F.Cu at (75.0, 45.0)
- added REF**: MountingHole_3.2mm_M3_Pad_Via, MountingHole:MountingHole_3.2mm_M3_Pad_Via, F.Cu at (155.0, 95.0)
- added REF**: OSHW-Logo2_7.3x6mm_SilkScreen, Symbol:OSHW-Logo2_7.3x6mm_SilkScreen, F.Cu at (98.4, 95.3)
- added REF**: MountingHole_3.2mm_M3_Pad_Via, MountingHole:MountingHole_3.2mm_M3_Pad_Via, F.Cu at (75.0, 95.0)
- added REF**: ESD-Logo_6.6x6mm_SilkScreen, Symbol:ESD-Logo_6.6x6mm_SilkScreen, F.Cu at (157.4, 54.8)
- added REF**: WEEE-Logo_4.2x6mm_SilkScreen, Symbol:WEEE-Logo_4.2x6mm_SilkScreen, F.Cu at (151.5, 54.7)
- added REF**: KiCad-Logo2_5mm_SilkScreen, Symbol:KiCad-Logo2_5mm_SilkScreen, F.Cu at (87.3, 94.9)
- J1: value OUT_12V_1 -> OUT_5V
- J10: value OUT_5V -> OUT_12V_5
- J11: value OUT_6V -> OUT_12V_6
- J12: value OUT_9V -> OUT_12V_7
- J13: value ISP -> OUT_12V_8; footprint Connector_PinHeader_2.54mm:PinHeader_2x03_P2.54mm_Vertical -> Connector_Wire:SolderWire-1.5sqmm_1x02_P6mm_D1.7mm_OD3mm
- J2: value OUT_12V_2 -> OUT_6V
- J3: value OUT_12V_3 -> OUT_9V
- J4: value OUT_12V_4 -> OUT_12V_1
- J5: value OUT_12V_5 -> OUT_12V_2
- J6: value OUT_12V_6 -> POWER_IN; footprint Connector_Wire:SolderWire-1.5sqmm_1x02_P6mm_D1.7mm_OD3mm -> Connector_Wire:SolderWire-1.5sqmm_1x05_P6mm_D1.7mm_OD3mm
- J7: value OUT_12V_7 -> GND; footprint Connector_Wire:SolderWire-1.5sqmm_1x02_P6mm_D1.7mm_OD3mm -> Connector_PinHeader_2.54mm:PinHeader_1x11_P2.54mm_Vertical
- J8: value OUT_12V_8 -> OUT_12V_3
- J9: value POWER_IN -> OUT_12V_4; footprint Connector_Wire:SolderWire-1.5sqmm_1x05_P6mm_D1.7mm_OD3mm -> Connector_Wire:SolderWire-1.5sqmm_1x02_P6mm_D1.7mm_OD3mm
- Q1, Q2, Q3, Q4, Q5, Q6, Q7, Q8: value BC807 -> IRLR024NTRPBF; footprint Package_TO_SOT_SMD:SOT-23_Handsoldering -> Package_TO_SOT_SMD:TO-252-3_TabPin2
- Q10, Q11, Q9: value BC817 -> IRLR024NTRPBF; footprint Package_TO_SOT_SMD:SOT-23_Handsoldering -> Package_TO_SOT_SMD:TO-252-3_TabPin2
- R1, R11, R12, R13, R14, R15, R16, R2, R3, R4, R5: value 1k -> 4k7
- R10, R19, R21, R6, R7, R8, R9: value 1k -> 470R
- R17, R18, R20: value 33R -> 470R
- R22: value 4k7 -> 470R
- moved J6 325.9 mm to (78.6, 77.9), turned to 90 degrees
- moved J1 317.9 mm to (84.0, 50.0), turned to 90 degrees
- moved J2 314.0 mm to (90.0, 50.0), turned to 90 degrees
- moved J3 304.7 mm to (96.0, 50.0), turned to 90 degrees
- moved J5 301.7 mm to (110.0, 50.0), turned to 90 degrees
- moved J7 295.6 mm to (104.3, 86.8), turned to 90 degrees
- moved J4 295.5 mm to (104.0, 50.0), turned to 90 degrees
- moved J8 291.0 mm to (116.0, 50.0), turned to 90 degrees
- moved Q5 280.2 mm to (114.7, 69.8), turned to -90 degrees
- moved Q7 279.4 mm to (129.0, 69.8), turned to -90 degrees
- moved R14 273.6 mm to (143.2, 62.0), turned to 180 degrees
- moved J10 268.4 mm to (128.0, 50.0), turned to 90 degrees
- moved J11 263.5 mm to (134.0, 50.0), turned to 90 degrees
- moved R20 260.4 mm to (143.8, 76.0)
- moved J12 258.9 mm to (140.0, 50.0), turned to 90 degrees
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Connections:
- J1 pad 2: +12V -> +5V
- J10 pad 2: +5V -> +12V
- J11 pad 2: +6V -> +12V
- J12 pad 2: +9V -> +12V
- J13 pad 1: /MISO -> Net-(J13-Pin_1)
- J13 pad 2: +5V -> +12V
- J2 pad 2: +12V -> +6V
- J3 pad 2: +12V -> +9V
- J6 pad 1: Net-(J6-Pin_1) -> GND
- J7 pad 1: Net-(J7-Pin_1) -> GND
- J7 pad 2: +12V -> GND
- J9 pad 1: GND -> Net-(J9-Pin_1)
- J9 pad 2: +5V -> +12V
- Q1 pad 1: Net-(Q1-B) -> Net-(Q1-G)
- Q1 pad 2: +5V -> Net-(J1-Pin_1)
- Q1 pad 3: Net-(Q1-C) -> GND
- Q10 pad 1: Net-(Q10-B) -> Net-(Q10-G)
- Q10 pad 2: GND -> Net-(J12-Pin_1)
- Q10 pad 3: Net-(Q10-C) -> GND
- Q11 pad 1: Net-(Q11-B) -> Net-(Q11-G)
- Q11 pad 2: GND -> Net-(J13-Pin_1)
- Q11 pad 3: Net-(Q11-C) -> GND
- Q2 pad 1: Net-(Q14-C) -> Net-(Q2-G)
- Q2 pad 2: +5V -> Net-(J2-Pin_1)
- Q2 pad 3: Net-(Q2-C) -> GND
- Q3 pad 1: Net-(Q16-C) -> Net-(Q3-G)
- Q3 pad 2: +5V -> Net-(J3-Pin_1)
- Q3 pad 3: Net-(Q3-C) -> GND
- Q4 pad 1: Net-(Q15-C) -> Net-(Q4-G)
- Q4 pad 2: +5V -> Net-(J4-Pin_1)
- Q4 pad 3: Net-(Q4-C) -> GND
- Q5 pad 1: Net-(Q37-C) -> Net-(Q5-G)
- Q5 pad 2: +5V -> Net-(J5-Pin_1)
- Q5 pad 3: Net-(Q5-C) -> GND
- Q6 pad 1: Net-(Q38-C) -> Net-(Q6-G)
- Q6 pad 2: +5V -> Net-(J8-Pin_1)
- Q6 pad 3: Net-(Q6-C) -> GND
- Q7 pad 1: Net-(Q39-C) -> Net-(Q7-G)
- Q7 pad 2: +5V -> Net-(J9-Pin_1)
- Q7 pad 3: Net-(Q7-C) -> GND
- Q8 pad 1: Net-(Q40-C) -> Net-(Q8-G)
- Q8 pad 2: +5V -> Net-(J10-Pin_1)
- Q8 pad 3: Net-(Q8-C) -> GND
- Q9 pad 1: Net-(Q9-B) -> Net-(Q9-G)
- Q9 pad 2: GND -> Net-(J11-Pin_1)
- Q9 pad 3: Net-(Q1-B) -> GND
- R1 pad 1: +5V -> Net-(Q1-G)
- R1 pad 2: Net-(Q29-B) -> GND
- R10 pad 1: /7SEG_4_1 -> /CTRL_9V
- R10 pad 2: Net-(Q40-B) -> Net-(Q3-G)
- R11 pad 1: /7SEG_1_1 -> Net-(Q6-G)
- R11 pad 2: Net-(Q14-B) -> GND
- R12 pad 1: /7SEG_2_1 -> Net-(Q7-G)
- R12 pad 2: Net-(Q16-B) -> GND
- R13 pad 1: /7SEG_3_2 -> Net-(Q8-G)
- R13 pad 2: Net-(Q34-B) -> GND
- R14 pad 1: /7SEG_4_2 -> Net-(Q9-G)
- R14 pad 2: Net-(Q36-B) -> GND
- R15 pad 1: /7SEG_1_2 -> Net-(Q10-G)
- R15 pad 2: Net-(Q10-B) -> GND
- R16 pad 1: /7SEG_2_2 -> Net-(Q11-G)
- R16 pad 2: Net-(Q12-B) -> GND
- R17 pad 1: Net-(U9-Q) -> /CTRL_12V_3
- R17 pad 2: /PWM_SIG_OUT_1 -> Net-(Q6-G)
- R18 pad 1: Net-(U10-Q) -> /CTRL_12V_4
- R18 pad 2: /PWM_SIG_OUT_2 -> Net-(Q7-G)
- R19 pad 1: Net-(D1-A) -> /CTRL_12V_5
- R19 pad 2: +5V -> Net-(Q8-G)
- R2 pad 1: +5V -> Net-(Q2-G)
- R2 pad 2: Net-(Q31-B) -> GND
- R20 pad 1: Net-(U11-Q) -> /CTRL_12V_6
- R20 pad 2: /PWM_SIG_OUT_3 -> Net-(Q9-G)
- R21 pad 1: Net-(D3-A) -> /CTRL_12V_7
- R21 pad 2: +5V -> Net-(Q10-G)
- R22 pad 1: Net-(Q17-G) -> /CTRL_12V_8
- R22 pad 2: GND -> Net-(Q11-G)
- R3 pad 1: +5V -> Net-(Q3-G)
- R3 pad 2: Net-(Q10-C) -> GND
- R4 pad 1: +5V -> Net-(Q4-G)
- R4 pad 2: Net-(Q12-C) -> GND
- R5 pad 1: +5V -> Net-(Q5-G)
- R5 pad 2: Net-(Q38-C) -> GND
- R6 pad 1: +5V -> /CTRL_12V_1
- R6 pad 2: Net-(Q40-C) -> Net-(Q4-G)
- R7 pad 1: +5V -> /CTRL_12V_2
- R7 pad 2: Net-(Q14-C) -> Net-(Q5-G)
- R8 pad 1: +5V -> /CTRL_5V
- R8 pad 2: Net-(Q16-C) -> Net-(Q1-G)
- R9 pad 1: /7SEG_3_1 -> /CTRL_6V
- R9 pad 2: Net-(Q38-B) -> Net-(Q2-G)
Routing:
- net +12V: track 0.00 -> 85.5 mm
- net +5V: track 0.00 -> 74.6 mm
- net /CTRL_5V: track 0.00 -> 54.3 mm
- net /CTRL_6V: track 0.00 -> 51.0 mm
- net /CTRL_9V: track 0.00 -> 46.4 mm
- net /CTRL_12V_1: track 0.00 -> 43.1 mm
- net /CTRL_12V_2: track 0.00 -> 38.0 mm
- net +9V: track 0.00 -> 37.4 mm
- net /CTRL_12V_3: track 0.00 -> 34.6 mm
- net /CTRL_12V_4: track 0.00 -> 29.2 mm
- net Net-(J13-Pin_1): track 0.00 -> 29.1 mm
- net +6V: track 0.00 -> 26.1 mm
- net /CTRL_12V_5: track 0.00 -> 25.3 mm
- net Net-(J12-Pin_1): track 0.00 -> 25.3 mm
- net Net-(J11-Pin_1): track 0.00 -> 24.8 mm
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- added copper zone on B.Cu, net GND
- added copper zone on F.Cu, net GND
Other:
- board size 260 x 140 mm -> 93 x 60 mm
- board text added: "12V"
- board text added: "5V"
- board text added: "6V"
- board text added: "9V"
- board text added: "GND"
- board text added: "Medium power distribution https://github.com/SniperCZE/astrobox"
