File: astrobox_medium/astrobox_power_mediumbox/astrobox_power_mediumbox.kicad_sch (KiCad schematic)
At the start: 310 parts, among them J1 OUT_12V_1, J10 OUT_5V, J11 OUT_6V, J12 OUT_9V, J13 ISP, J14 TO_CONTROL, J15 TO_OUTPUT, J2 OUT_12V_2, J3 OUT_12V_3, J4 OUT_12V_4, J5 OUT_12V_5, J6 OUT_12V_6, J7 OUT_12V_7, J8 OUT_12V_8, J9 POWER_IN, Q1 BC807, Q10 BC817, Q11 BC817, Q12 BC817, Q13 BC817, Q14 BC817, Q15 BC817, Q16 BC817, Q17 IRLZ34N, Q18 IRLZ34N, Q19 IRLZ34N, Q2 BC807, Q20 IRLZ34N, Q21 IRLZ34N, Q22 IRLZ34N, Q23 IRLZ34N, Q24 IRLZ34N, Q25 BC807, Q26 BC807, Q27 BC807, Q28 BC807, Q29 BC807, Q3 BC807, Q30 BC807, Q31 BC807, Q33 BC817, Q34 BC817, Q35 BC817, Q36 BC817, Q37 BC817, Q38 BC817, Q39 BC817, Q4 BC807, Q40 BC817, Q41 IRLZ34N, Q42 IRLZ34N, Q43 IRLZ34N, Q44 BC807, Q5 BC807, Q6 BC807, Q7 BC807, Q8 BC807, Q9 BC817, SW1 PWM_ENB_1, SW10 ENB_9V, SW11 ENB_12V_6, SW12 ENB_6V, SW13 ENB_12V_5, SW14 ENB_5V, SW15 ENB_12V_4, SW16 PWM_ENB_5, SW17 PWM_ENB_6, SW18 PWM_ENB_7, SW19 PWM_ENB_8, SW2 PWM_ENB_2, SW3 PWM_ENB_3, SW4 PWM_ENB_4, SW5 ENB_12V_3, SW6 ENB_12V_2, SW7 ENB_12V_8, SW8 ENB_12V_1, SW9 ENB_12V_7, U1 DA56-11EWA, U10 NE555P, U11 NE555P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

Commit message: medium astrobox in multiple boards
Parts:
- removed J14: TO_CONTROL, Connector_PinHeader_2.54mm:PinHeader_1x29_P2.54mm_Vertical, symbol Connector_Generic:Conn_01x29
- removed J15: TO_OUTPUT, Connector_PinHeader_2.54mm:PinHeader_1x29_P2.54mm_Vertical, symbol Connector_Generic:Conn_01x29
- removed Q17, Q18, Q19, Q20, Q21, Q22, Q23, Q24, Q41, Q42, Q43: IRLZ34N, Package_TO_SOT_THT:TO-220-3_Vertical, symbol Transistor_FET:IRLZ34N
- added Q17, Q18, Q19, Q20, Q21, Q22, Q23, Q24, Q32, Q41, Q42: IRLR024NTRPBF, Package_TO_SOT_SMD:TO-252-3_TabPin2, symbol Transistor_FET:Q_NMOS_GSD
Connections:
- net GND: now also Q17.3 (D), Q18.3 (D), Q19.3 (D), Q20.3 (D), Q21.3 (D), Q22.3 (D), Q23.3 (D), Q24.3 (D), Q32.2 (S), Q41.2 (S), Q42.2 (S)
- net at R23.1, R34.2: now also Q18.1 (G)
- net at J2.1 (Pin_1): now also Q18.2 (S)
- net at R26.1, R37.2: now also Q21.1 (G)
- net at R29.1, R40.2: now also Q24.1 (G)
- net at R27.1, R38.2: now also Q22.1 (G)
- net at R57.1, R64.2: now also Q41.1 (G)
- net at J10.1 (Pin_1): now also Q41.3 (D)
- net at R24.1, R35.2: now also Q19.1 (G)
- net at R58.1, R65.2: now also Q32.1 (G)
- net at R59.1, R66.2: now also Q42.1 (G)
- net at J12.1 (Pin_1): now also Q42.3 (D)
- net at R28.1, R39.2: now also Q23.1 (G)
- net at R22.1, R33.2: now also Q17.1 (G)
- net at R25.1, R36.2: now also Q20.1 (G)
- net at J1.1 (Pin_1): now also Q17.2 (S)
- net at J7.1 (Pin_1): now also Q23.2 (S)
- net at J6.1 (Pin_1): now also Q22.2 (S)
- net at J11.1 (Pin_1): now also Q32.3 (D)
- net at J8.1 (Pin_1): now also Q24.2 (S)
- net at J3.1 (Pin_1): now also Q19.2 (S)
- net at J5.1 (Pin_1): now also Q21.2 (S)
- net at J4.1 (Pin_1): now also Q20.2 (S)

Commit message: astrobox medium final pcb
Parts:
- removed C1, C11, C13, C14, C15, C16, C17, C18, C19, C2, C20, C21, C22, C23, C24, C25, C26, C27, C28, C29, C3, C31, C33, C35, C37, C38, C39, C4, C5, C7, C9: 100n, Capacitor_SMD:C_1206_3216Metric_Pad1.33x1.80mm_HandSolder, symbol Device:C
- removed C10, C12, C30, C32, C34, C36, C6, C8: 1n, Capacitor_SMD:C_1206_3216Metric_Pad1.33x1.80mm_HandSolder, symbol Device:C
- removed D1, D14, D15, D16, D17, D2, D20, D21, D22, D23, D3, D4, D5, D6, D7, D8: 1N4007, Diode_SMD:D_SMA-SMB_Universal_Handsoldering, symbol Device:D
- removed D10: PWM_ENB_2, LED_THT:LED_D5.0mm, symbol Device:LED
- removed D11: PWM_ENB_3, LED_THT:LED_D5.0mm, symbol Device:LED
- removed D12: PWM_ENB_4, LED_THT:LED_D5.0mm, symbol Device:LED
- removed D13: ENB_12V_3, LED_THT:LED_D5.0mm, symbol Device:LED
- removed D18: ENB_12V_2, LED_THT:LED_D5.0mm, symbol Device:LED
- removed D19: ENB_12V_8, LED_THT:LED_D5.0mm, symbol Device:LED
- removed D24: ENB_12V_1, LED_THT:LED_D5.0mm, symbol Device:LED
- removed D25: ENB_12V_7, LED_THT:LED_D5.0mm, symbol Device:LED
- removed D26: ENB_9V, LED_THT:LED_D5.0mm, symbol Device:LED
- removed D27: ENB_12V_6, LED_THT:LED_D5.0mm, symbol Device:LED
- removed D28: ENB_6V, LED_THT:LED_D5.0mm, symbol Device:LED
- removed D29: ENB_12V_5, LED_THT:LED_D5.0mm, symbol Device:LED
- removed D30: ENB_5V, LED_THT:LED_D5.0mm, symbol Device:LED
- removed D31: ENB_12V_4, LED_THT:LED_D5.0mm, symbol Device:LED
- removed D32: PWM_ENB_5, LED_THT:LED_D5.0mm, symbol Device:LED
- removed D33: PWM_ENB_6, LED_THT:LED_D5.0mm, symbol Device:LED
- removed D34: PWM_ENB_7, LED_THT:LED_D5.0mm, symbol Device:LED
- removed D35: PWM_ENB_8, LED_THT:LED_D5.0mm, symbol Device:LED
- removed D9: PWM_ENB_1, LED_THT:LED_D5.0mm, symbol Device:LED
- removed J13: ISP, Connector_PinHeader_2.54mm:PinHeader_2x03_P2.54mm_Vertical, symbol Connector_Generic:Conn_02x03_Odd_Even
- removed Q1, Q2, Q25, Q26, Q27, Q28, Q29, Q3, Q30, Q31, Q4, Q44, Q5, Q6, Q7, Q8: BC807, Package_TO_SOT_SMD:SOT-23_Handsoldering, symbol Transistor_BJT:BC807
- removed Q10, Q11, Q12, Q13, Q14, Q15, Q16, Q33, Q34, Q35, Q36, Q37, Q38, Q39, Q40, Q9: BC817, Package_TO_SOT_SMD:SOT-23_Handsoldering, symbol Transistor_BJT:BC817
- removed R1, R10, R11, R12, R13, R14, R15, R16, R19, R2, R21, R3, R31, R32, R4, R41, R42, R43, R44, R45, R46, R47, R48, R49, R5, R50, R51, R52, R53, R54, R55, R56, R6, R60, R61, R62, R63, R7, R8, R81, R83, R85, R86, R9, R92, R93, R94, R95: 1k, Resistor_SMD:R_1206_3216Metric_Pad1.30x1.75mm_HandSolder, symbol Device:R
- removed R100, R101, R102, R103, R104, R105, R67, R68, R69, R70, R71, R72, R73, R74, R75, R76, R77, R78, R87, R88, R89, R90, R91, R96, R97, R98, R99: 330R, Resistor_SMD:R_1206_3216Metric_Pad1.30x1.75mm_HandSolder, symbol Device:R
- removed R106, R107, R108, R109, R110, R111, R112, R113, R114, R115, R116, R117, R118, R119, R120, R121: 100k, Resistor_SMD:R_1206_3216Metric_Pad1.30x1.75mm_HandSolder, symbol Device:R
- removed R17, R18, R20, R30, R79, R80, R82, R84: 33R, Resistor_SMD:R_1206_3216Metric_Pad1.30x1.75mm_HandSolder, symbol Device:R
- removed RV1: PWM_SET_1, Connector_Wire:SolderWire-1sqmm_1x03_P5.4mm_D1.4mm_OD2.7mm, symbol Device:R_Potentiometer
- removed RV2: PWM_SET_2, Connector_Wire:SolderWire-1sqmm_1x03_P5.4mm_D1.4mm_OD2.7mm, symbol Device:R_Potentiometer
- removed RV3: PWM_SET_3, Connector_Wire:SolderWire-1sqmm_1x03_P5.4mm_D1.4mm_OD2.7mm, symbol Device:R_Potentiometer
- removed RV4: PWM_SET_4, Connector_Wire:SolderWire-1sqmm_1x03_P5.4mm_D1.4mm_OD2.7mm, symbol Device:R_Potentiometer
- removed RV5: PWM_SET_5, Connector_Wire:SolderWire-1sqmm_1x03_P5.4mm_D1.4mm_OD2.7mm, symbol Device:R_Potentiometer
- removed RV6: PWM_SET_6, Connector_Wire:SolderWire-1sqmm_1x03_P5.4mm_D1.4mm_OD2.7mm, symbol Device:R_Potentiometer
- removed RV7: PWM_SET_7, Connector_Wire:SolderWire-1sqmm_1x03_P5.4mm_D1.4mm_OD2.7mm, symbol Device:R_Potentiometer
- removed RV8: PWM_SET_8, Connector_Wire:SolderWire-1sqmm_1x03_P5.4mm_D1.4mm_OD2.7mm, symbol Device:R_Potentiometer
- removed SW1: PWM_ENB_1, Connector_Wire:SolderWire-1sqmm_1x02_P5.4mm_D1.4mm_OD2.7mm, symbol Switch:SW_Push
- removed SW10: ENB_9V, Connector_Wire:SolderWire-1sqmm_1x02_P5.4mm_D1.4mm_OD2.7mm, symbol Switch:SW_Push
- removed SW11: ENB_12V_6, Connector_Wire:SolderWire-1sqmm_1x02_P5.4mm_D1.4mm_OD2.7mm, symbol Switch:SW_Push
- removed SW12: ENB_6V, Connector_Wire:SolderWire-1sqmm_1x02_P5.4mm_D1.4mm_OD2.7mm, symbol Switch:SW_Push
- removed SW13: ENB_12V_5, Connector_Wire:SolderWire-1sqmm_1x02_P5.4mm_D1.4mm_OD2.7mm, symbol Switch:SW_Push
- removed SW14: ENB_5V, Connector_Wire:SolderWire-1sqmm_1x02_P5.4mm_D1.4mm_OD2.7mm, symbol Switch:SW_Push
- removed SW15: ENB_12V_4, Connector_Wire:SolderWire-1sqmm_1x02_P5.4mm_D1.4mm_OD2.7mm, symbol Switch:SW_Push
- removed SW16: PWM_ENB_5, Connector_Wire:SolderWire-1sqmm_1x02_P5.4mm_D1.4mm_OD2.7mm, symbol Switch:SW_Push
- removed SW17: PWM_ENB_6, Connector_Wire:SolderWire-1sqmm_1x02_P5.4mm_D1.4mm_OD2.7mm, symbol Switch:SW_Push
- removed SW18: PWM_ENB_7, Connector_Wire:SolderWire-1sqmm_1x02_P5.4mm_D1.4mm_OD2.7mm, symbol Switch:SW_Push
- removed SW19: PWM_ENB_8, Connector_Wire:SolderWire-1sqmm_1x02_P5.4mm_D1.4mm_OD2.7mm, symbol Switch:SW_Push
- removed SW2: PWM_ENB_2, Connector_Wire:SolderWire-1sqmm_1x02_P5.4mm_D1.4mm_OD2.7mm, symbol Switch:SW_Push
- removed SW3: PWM_ENB_3, Connector_Wire:SolderWire-1sqmm_1x02_P5.4mm_D1.4mm_OD2.7mm, symbol Switch:SW_Push
- removed SW4: PWM_ENB_4, Connector_Wire:SolderWire-1sqmm_1x02_P5.4mm_D1.4mm_OD2.7mm, symbol Switch:SW_Push
- removed SW5: ENB_12V_3, Connector_Wire:SolderWire-1sqmm_1x02_P5.4mm_D1.4mm_OD2.7mm, symbol Switch:SW_Push
- removed SW6: ENB_12V_2, Connector_Wire:SolderWire-1sqmm_1x02_P5.4mm_D1.4mm_OD2.7mm, symbol Switch:SW_Push
- removed SW7: ENB_12V_8, Connector_Wire:SolderWire-1sqmm_1x02_P5.4mm_D1.4mm_OD2.7mm, symbol Switch:SW_Push
- removed SW8: ENB_12V_1, Connector_Wire:SolderWire-1sqmm_1x02_P5.4mm_D1.4mm_OD2.7mm, symbol Switch:SW_Push
- removed SW9: ENB_12V_7, Connector_Wire:SolderWire-1sqmm_1x02_P5.4mm_D1.4mm_OD2.7mm, symbol Switch:SW_Push
- removed U1, U2, U3, U4, U5, U6, U7, U8: DA56-11EWA, Display_7Segment:DA56-11SURKWA, symbol Display_Character:DA56-11EWA
- removed U10, U11, U14, U23, U24, U25, U26, U9: NE555P, Package_SO:SOIC-8_5.3x6.2mm_P1.27mm, symbol Timer:NE555P
- removed U12, U13, U20, U22, U27, U30: 74LS08, Package_SO:SO-14_3.9x8.65mm_P1.27mm, symbol 74xx:74LS08
- removed U15, U16: 74LS32, Package_DIP:DIP-14_W7.62mm_Socket, symbol 74xx:74LS32
- removed U17, U18: 74AHC04, Package_SO:SO-14_3.9x8.65mm_P1.27mm, symbol 74xx:74AHC04
- removed U19: 74LS47, Package_DIP:DIP-16_W7.62mm_Socket, symbol 74xx:74LS47
- removed U21, U29: 74HC4051, Package_SO:SOIC-16_3.9x9.9mm_P1.27mm, symbol 74xx:74HC4051
- removed U28: ATmega16A-M, Package_QFP:TQFP-44-1EP_10x10mm_P0.8mm_EP4.5x4.5mm, symbol MCU_Microchip_ATmega:ATmega16A-M
- added J14: +5V, Connector_PinHeader_2.54mm:PinHeader_1x11_P2.54mm_Vertical, symbol Connector_Generic:Conn_01x11
- added J15: Control, Connector_PinHeader_2.54mm:PinHeader_1x11_P2.54mm_Vertical, symbol Connector_Generic:Conn_01x11
- added J7: GND, Connector_PinHeader_2.54mm:PinHeader_1x11_P2.54mm_Vertical, symbol Connector_Generic:Conn_01x11
- renumbered J10 to J1, J5 to J10, J6 to J11, J7 to J12, J8 to J13, J11 to J2, J12 to J3, J1 to J4, J2 to J5, J9 to J6, J3 to J8, J4 to J9, Q41 to Q1, Q23 to Q10, Q24 to Q11, Q32 to Q2, Q42 to Q3, Q17 to Q4, Q18 to Q5, Q19 to Q6, Q20 to Q7, Q21 to Q8, Q22 to Q9, R57 to R1, R66 to R10, R24 to R11, R25 to R12, R26 to R13, R27 to R14, R28 to R15, R29 to R16, R35 to R17, R36 to R18, R37 to R19, R58 to R2, R38 to R20, R39 to R21, R40 to R22, R59 to R3, R22 to R4, R23 to R5, R33 to R6, R34 to R7, R64 to R8, R65 to R9
Connections:
- net +12V: now also J6.2 (Pin_2); no longer J6.5 (Pin_5)
- net +5V: now also J6.5 (Pin_5), J14.1 (Pin_1), J14.10 (Pin_10), J14.11 (Pin_11), J14.2 (Pin_2), J14.3 (Pin_3), J14.4 (Pin_4), J14.5 (Pin_5), J14.6 (Pin_6), J14.7 (Pin_7), J14.8 (Pin_8), J14.9 (Pin_9); no longer J6.2 (Pin_2)
- net +6V: now also J6.4 (Pin_4); no longer J6.3 (Pin_3)
- net +9V: now also J6.3 (Pin_3); no longer J6.4 (Pin_4)
- net GND: now also Q1.3 (D), Q2.3 (D), Q3.3 (D), J7.1 (Pin_1), J7.10 (Pin_10), J7.11 (Pin_11), J7.2 (Pin_2), J7.3 (Pin_3), J7.4 (Pin_4), J7.5 (Pin_5), J7.6 (Pin_6), J7.7 (Pin_7), J7.8 (Pin_8), J7.9 (Pin_9); no longer Q1.2 (S), Q2.2 (S), Q3.2 (S)
- net CTRL_12V_7: now reaches R21.1
- net CTRL_12V_7: now also J15.10 (Pin_10)
- net CTRL_12V_6: now reaches R20.1
- net CTRL_12V_6: now also J15.9 (Pin_9)
- net CTRL_12V_5: now reaches R19.1
- net CTRL_12V_5: now also J15.8 (Pin_8)
- net CTRL_12V_3: now reaches R17.1
- net CTRL_12V_3: now also J15.6 (Pin_6)
- net CTRL_12V_1: now reaches R6.1
- net CTRL_12V_1: now also J15.4 (Pin_4)
- net at J3.1 (Pin_1): now also Q3.2 (S); no longer Q3.3 (D)
- net CTRL_12V_2: now reaches R7.1
- net CTRL_12V_2: now also J15.5 (Pin_5)
- net CTRL_12V_4: now reaches R18.1
- net CTRL_12V_4: now also J15.7 (Pin_7)
- net CTRL_12V_8: now reaches R22.1
- net CTRL_12V_8: now also J15.11 (Pin_11)
- net at J1.1 (Pin_1): now also Q1.2 (S); no longer Q1.3 (D)
- net at J2.1 (Pin_1): now also Q2.2 (S); no longer Q2.3 (D)
- net ENABLE_5V renamed CTRL_5V
- net CTRL_5V: now also J15.1 (Pin_1)
- net ENABLE_6V renamed CTRL_6V
- net CTRL_6V: now also J15.2 (Pin_2)
- net ENABLE_9V renamed CTRL_9V
- net CTRL_9V: now also J15.3 (Pin_3)
Other:
- moved on the sheet: J1, J10, J11, J12, J13, J2, J3, J4, J5, J6, J8, J9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
