File: astrobox_medium/control_board/control_board.kicad_pcb (KiCad board)
At the start: 2 copper layers, 46 x 100 mm, 70 parts, among them J1 ISP, J2 Output, Q1 BC817, Q10 BC817, Q11 BC817, Q12 BC817, Q13 BC817, Q14 BC817, Q2 BC817, Q3 BC817, Q4 BC817, Q5 BC817, Q6 BC817, Q7 BC817, Q8 BC817, Q9 BC817, SW1 Enable, SW2 Enbl PWM, U1 DA56-11EWA, U2 ATmega8535-16A, U3 74LS14

Commit message: Control board update
Parts:
- R18, R19: value 10k -> 1k
- SW2: value Enbl PWM -> Enable PWM
Connections:
- D1 pad 2: Net-(D1-A) -> /ENB
- D2 pad 2: Net-(D2-A) -> /ENB_PWM
- SW1 pad 2: Net-(D1-A) -> GND
- SW2 pad 2: Net-(D2-A) -> GND
Routing:
- net /ENB_PWM: track 3.84 -> 40.5 mm, vias 0 -> 1
- net /ENB: track 3.12 -> 24.4 mm, vias 0 -> 1
- net Net-(D2-A): track 6.25 -> 0.00 mm
- net Net-(D1-A): track 6.18 -> 0.00 mm
