File: astrobox_medium/control_board/control_board.kicad_sch (KiCad schematic)
At the start: 65 parts, among them J1 ISP, J2 Conn_01x03, Q1 BC817, Q10 BC817, Q11 BC817, Q12 BC817, Q13 BC817, Q14 BC817, Q2 BC817, Q3 BC817, Q4 BC817, Q5 BC817, Q6 BC817, Q7 BC817, Q8 BC817, Q9 BC817, SW1 SW_SPST, SW2 SW_SPST, U1 ATmega8535-16A, U2 DA56-11EWA, U3 74LS14

Commit message: astrobox medium final pcb
Parts:
- removed C1: 100n, symbol Device:C
- removed D1, D2: 1N4007, Diode_THT:D_DO-41_SOD81_P10.16mm_Horizontal, symbol Diode:1N4007
- removed J2: Conn_01x03, symbol Connector_Generic:Conn_01x03
- removed R31, R34: 10k, symbol Device:R
- added C5: 100n, Capacitor_SMD:C_1206_3216Metric_Pad1.33x1.80mm_HandSolder, symbol Device:C
- added J2: Output, Connector_Wire:SolderWire-1.5sqmm_1x05_P6mm_D1.7mm_OD3mm, symbol Connector_Generic:Conn_01x05
- added R15, R19: 10k, Resistor_SMD:R_1206_3216Metric_Pad1.30x1.75mm_HandSolder, symbol Device:R
- C1: renamed from C2; footprint (none) -> Capacitor_SMD:C_1206_3216Metric_Pad1.33x1.80mm_HandSolder
- C2: renamed from C3; footprint (none) -> Capacitor_SMD:C_1206_3216Metric_Pad1.33x1.80mm_HandSolder
- C3: renamed from C4; footprint (none) -> Capacitor_SMD:C_1206_3216Metric_Pad1.33x1.80mm_HandSolder
- C4: renamed from C5; footprint (none) -> Capacitor_SMD:C_1206_3216Metric_Pad1.33x1.80mm_HandSolder
- D1: renamed from D3; value LED -> Ind E; footprint (none) -> LED_THT:LED_D5.0mm
- D2: renamed from D4; value LED -> Ind E PWM; footprint (none) -> LED_THT:LED_D5.0mm
- J1: footprint (none) -> Connector_PinHeader_2.54mm:PinHeader_2x03_P2.54mm_Vertical
- R1: renamed from R12; footprint (none) -> Resistor_SMD:R_1206_3216Metric_Pad1.30x1.75mm_HandSolder
- R10: renamed from R7; footprint (none) -> Resistor_SMD:R_1206_3216Metric_Pad1.30x1.75mm_HandSolder
- R11: renamed from R9; footprint (none) -> Resistor_SMD:R_1206_3216Metric_Pad1.30x1.75mm_HandSolder
- R12: renamed from R6; footprint (none) -> Resistor_SMD:R_1206_3216Metric_Pad1.30x1.75mm_HandSolder
- R13: renamed from R5; footprint (none) -> Resistor_SMD:R_1206_3216Metric_Pad1.30x1.75mm_HandSolder
- R14, R25: footprint (none) -> Resistor_SMD:R_1206_3216Metric_Pad1.30x1.75mm_HandSolder
- R16: renamed from R32; footprint (none) -> Resistor_SMD:R_1206_3216Metric_Pad1.30x1.75mm_HandSolder
- R17: renamed from R15; footprint (none) -> Resistor_SMD:R_1206_3216Metric_Pad1.30x1.75mm_HandSolder
- R18: renamed from R33; footprint (none) -> Resistor_SMD:R_1206_3216Metric_Pad1.30x1.75mm_HandSolder
- R2: renamed from R4; footprint (none) -> Resistor_SMD:R_1206_3216Metric_Pad1.30x1.75mm_HandSolder
- R20: renamed from R16; footprint (none) -> Resistor_SMD:R_1206_3216Metric_Pad1.30x1.75mm_HandSolder
- R21: renamed from R17; footprint (none) -> Resistor_SMD:R_1206_3216Metric_Pad1.30x1.75mm_HandSolder
- R22: renamed from R19; footprint (none) -> Resistor_SMD:R_1206_3216Metric_Pad1.30x1.75mm_HandSolder
- R23: renamed from R21; footprint (none) -> Resistor_SMD:R_1206_3216Metric_Pad1.30x1.75mm_HandSolder
- R24: renamed from R23; footprint (none) -> Resistor_SMD:R_1206_3216Metric_Pad1.30x1.75mm_HandSolder
- R26: renamed from R27; footprint (none) -> Resistor_SMD:R_1206_3216Metric_Pad1.30x1.75mm_HandSolder
- R27: renamed from R30; footprint (none) -> Resistor_SMD:R_1206_3216Metric_Pad1.30x1.75mm_HandSolder
- R28: renamed from R13; footprint (none) -> Resistor_SMD:R_1206_3216Metric_Pad1.30x1.75mm_HandSolder
- R29: renamed from R18; footprint (none) -> Resistor_SMD:R_1206_3216Metric_Pad1.30x1.75mm_HandSolder
- R3: renamed from R8; footprint (none) -> Resistor_SMD:R_1206_3216Metric_Pad1.30x1.75mm_HandSolder
- R30: renamed from R20; footprint (none) -> Resistor_SMD:R_1206_3216Metric_Pad1.30x1.75mm_HandSolder
- R31: renamed from R22; footprint (none) -> Resistor_SMD:R_1206_3216Metric_Pad1.30x1.75mm_HandSolder
- R32: renamed from R24; footprint (none) -> Resistor_SMD:R_1206_3216Metric_Pad1.30x1.75mm_HandSolder
- R33: renamed from R26; footprint (none) -> Resistor_SMD:R_1206_3216Metric_Pad1.30x1.75mm_HandSolder
- R34: renamed from R29; footprint (none) -> Resistor_SMD:R_1206_3216Metric_Pad1.30x1.75mm_HandSolder
- R4: renamed from R10; footprint (none) -> Resistor_SMD:R_1206_3216Metric_Pad1.30x1.75mm_HandSolder
- R5: renamed from R1; footprint (none) -> Resistor_SMD:R_1206_3216Metric_Pad1.30x1.75mm_HandSolder
- R6: renamed from R3; footprint (none) -> Resistor_SMD:R_1206_3216Metric_Pad1.30x1.75mm_HandSolder
- R7: renamed from R28; footprint (none) -> Resistor_SMD:R_1206_3216Metric_Pad1.30x1.75mm_HandSolder
- R8: renamed from R11; footprint (none) -> Resistor_SMD:R_1206_3216Metric_Pad1.30x1.75mm_HandSolder
- R9: renamed from R2; footprint (none) -> Resistor_SMD:R_1206_3216Metric_Pad1.30x1.75mm_HandSolder
- RV1: value R_Potentiometer -> PWM SET; footprint (none) -> Connector_Wire:SolderWire-1sqmm_1x03_P5.4mm_D1.4mm_OD2.7mm
- SW1: value SW_SPST -> Enable; footprint (none) -> Connector_Wire:SolderWire-1sqmm_1x02_P5.4mm_D1.4mm_OD2.7mm
- SW2: value SW_SPST -> Enable PWM; footprint (none) -> Connector_Wire:SolderWire-1sqmm_1x02_P5.4mm_D1.4mm_OD2.7mm
- U3: footprint (none) -> Package_SO:SO-14_3.9x8.65mm_P1.27mm
- renumbered Q7 to Q1, Q3 to Q2, Q4 to Q3, Q5 to Q4, Q2 to Q5, Q1 to Q6, Q6 to Q7, U2 to U1, U1 to U2
Connections:
- net +5V: now also C4.1, R16.1, RV1.1, U3.14 (VCC), J2.5 (Pin_5), R15.2
- net DIG1_A: now also R14.1, U2.32 (PA5); no longer U2.36 (PA1)
- net DIG1_B: now also R13.1, U2.33 (PA4); no longer U2.35 (PA2)
- net DIG1_C: now also R12.1, U2.36 (PA1); no longer U2.34 (PA3)
- net DIG1_D: now also R11.1, U2.35 (PA2); no longer U2.33 (PA4)
- net DIG1_E: now also R10.1, U2.34 (PA3); no longer U2.32 (PA5)
- net DIG1_F: now also R9.1, U2.30 (PA7); no longer U2.31 (PA6)
- net DIG1_G: now also R8.1, U2.31 (PA6); no longer U2.30 (PA7)
- net GND: now also C2.2, C3.2, C4.2, J1.5 (Pin_5), R17.2, R20.2, RV1.3, U3.7 (GND), C5.2, J2.1 (Pin_1); no longer J1.4 (Pin_4)
- net MISO: now also J1.1 (Pin_1); no longer J1.2 (Pin_2)
- net MOSI: now also J1.2 (Pin_2); no longer J1.3 (Pin_3)
- net OUTPUT: now also J2.4 (Pin_4)
- net PWM_SET: now also RV1.2, C5.1
- net RST: now also J1.3 (Pin_3); no longer J1.1 (Pin_1)
- net SCK: now also J1.4 (Pin_4); no longer J1.5 (Pin_5)
- net at D2.1 (K): now also R20.1
- net at D2.2 (A): now also SW2.2 (B)
- net at C3.1: now also U3.3, R19.1
- net DIG2_D: now reaches R31.1
- net DIG2_D: now also U2.11 (PD2)
- net at C2.1: now also R18.2, U3.1
- net ENB_PWM: now reaches U3.4
- net ENB_PWM: now also U2.40 (PB0)
- net DIG2_F: now reaches R29.1
- net DIG2_F: now also U2.15 (PD6)
- net DIG2_C: now reaches R32.1
- net DIG2_C: now also U2.10 (PD1)
- net ENB: now reaches U3.2
- net ENB: now also U2.41 (PB1)
- net at R18.1: now also SW1.1 (A), R15.1
- net at SW2.1 (A): now also R16.2, R19.2
- net DIG2_A: now reaches R34.1
- net DIG2_A: now also U2.12 (PD3)
- net at SW1.2 (B): now also D1.2 (A)
- net DIG2_B: now reaches R33.1
- net DIG2_B: now also U2.14 (PD5)
- net at R17.1: now also D1.1 (K)
- net DIG2_E: now reaches R30.1
- net DIG2_E: now also U2.13 (PD4)
- net DIG2_G: now reaches U2.16 (PD7)
- net DIG2_G: now also R28.1
- net SCL: now reaches U2.19 (PC0)
- net SCL: now also J2.3 (Pin_3)
- net SDA: now reaches U2.20 (PC1)
- net SDA: now also J2.2 (Pin_2)
Other:
- moved on the sheet: C2, C3, C4, D1, D2, Q10, Q11, Q12, Q13, Q14, Q8, Q9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

Commit message: Control board update
Parts:
- R18, R19: value 10k -> 1k
Connections:
- net ENB: now also D1.2 (A)
- net ENB_PWM: now also D2.2 (A)
- net GND: now also SW1.2 (B), SW2.2 (B)
Other:
- moved on the sheet: C2, C3, D1, D2, R17, R18, R19, R20, U3A, U3B
